File: hardware/can-io-module/can-io-module.kicad_sch (KiCad schematic)
At the start: 0 parts

Commit message: feat: generate connected CAN IO schematic and SWD header
Parts:
- added C1: 10uF 50V input, DIY_DASH:1210, symbol Connector_Generic:Conn_01x02
- added C101, C102, C103, C104, C105, C106, C107, C108: 100nF ADC filter, DIY_DASH:0603, symbol Connector_Generic:Conn_01x02
- added C2: 22uF 10V buck output, DIY_DASH:1206, symbol Connector_Generic:Conn_01x02
- added C3: 4.7uF 10V 3V3 bulk, DIY_DASH:0805, symbol Connector_Generic:Conn_01x02
- added C4: 100nF U1 VDD1, DIY_DASH:0603, symbol Connector_Generic:Conn_01x02
- added C5: 100nF U1 VDD2, DIY_DASH:0603, symbol Connector_Generic:Conn_01x02
- added C6: 100nF U1 VDDA, DIY_DASH:0603, symbol Connector_Generic:Conn_01x02
- added D1: SMBJ33A, DIY_DASH:SMB_DO-214AA, symbol Connector_Generic:Conn_01x02
- added D2: Buck catch diode 60V, DIY_DASH:SMA_DO-214AC, symbol Connector_Generic:Conn_01x02
- added D3: CAN TVS, DIY_DASH:SOT23, symbol Connector_Generic:Conn_01x02
- added D4: K-line TVS 24V, DIY_DASH:SMA_DO-214AC, symbol Connector_Generic:Conn_01x02
- added D5: Flex TVS 5V, DIY_DASH:SOD323, symbol Connector_Generic:Conn_01x02
- added D6: AOUT1 ESD, DIY_DASH:SOD323, symbol Connector_Generic:Conn_01x02
- added D7: AOUT2 ESD, DIY_DASH:SOD323, symbol Connector_Generic:Conn_01x02
- added F1: 1A input fuse, DIY_DASH:NANO2_2410, symbol Connector_Generic:Conn_01x02
- added F2: 250mA resettable sensor fuse, DIY_DASH:1206, symbol Connector_Generic:Conn_01x02
- added FB1: 600R ferrite VDDA, DIY_DASH:0603, symbol Connector_Generic:Conn_01x02
- added J1: ECU_FCI_24P_RightAngle, DIY_DASH:ECU_FCI_24P_RightAngle, symbol Connector_Generic:Conn_01x24
- added J2: SWD_1x05_P2.54mm_DNP, Connector_PinHeader_2.54mm:PinHeader_1x05_P2.54mm_Vertical, symbol Connector_Generic:Conn_01x05
- added JP1: 120R CAN termination, DIY_DASH:0603, symbol Connector_Generic:Conn_01x02
- added L1: 22uH buck inductor, DIY_DASH:5.5x5.5mm, symbol Connector_Generic:Conn_01x02
- added L2: CAN common-mode choke, DIY_DASH:1812_common-mode, symbol Connector_Generic:Conn_01x04
- added Q1: 60V P-channel reverse polarity, DIY_DASH:PowerPAK_SO-8, symbol Connector_Generic:Conn_01x04
- added Q4: 60V logic N-MOS RELAY1, DIY_DASH:LFPAK56, symbol Connector_Generic:Conn_01x08
- added Q5: 60V logic N-MOS RELAY2, DIY_DASH:LFPAK56, symbol Connector_Generic:Conn_01x08
- added R1: 1.00k 1% excitation, DIY_DASH:0603, symbol Connector_Generic:Conn_01x02
- added R10: 100k BOOT0 pull-down, DIY_DASH:0603, symbol Connector_Generic:Conn_01x02
- added R101, R102, R103, R104, R105, R106, R107, R108: 10.0k 1% AIN series, DIY_DASH:0603, symbol Connector_Generic:Conn_01x02
- added R111, R112, R113, R114, R115, R116, R117, R118: 15.0k 1% AIN lower, DIY_DASH:0603, symbol Connector_Generic:Conn_01x02
- added R2: 4.70k 1% excitation, DIY_DASH:0603, symbol Connector_Generic:Conn_01x02
- added R3, R4: 100k mux enable safe-state, DIY_DASH:0603, symbol Connector_Generic:Conn_01x02
- added R5, R6: 100k relay gate pull-down, DIY_DASH:0603, symbol Connector_Generic:Conn_01x02
- added R7: 220R AOUT1 isolation, DIY_DASH:0603, symbol Connector_Generic:Conn_01x02
- added R8: 220R AOUT2 isolation, DIY_DASH:0603, symbol Connector_Generic:Conn_01x02
- added R9: 10k NRST pull-up, DIY_DASH:0603, symbol Connector_Generic:Conn_01x02
- added TP1: SWDIO, DIY_DASH:Test_pad, symbol Connector_Generic:Conn_01x01
- added TP2: SWCLK, DIY_DASH:Test_pad, symbol Connector_Generic:Conn_01x01
- added TP3: NRST, DIY_DASH:Test_pad, symbol Connector_Generic:Conn_01x01
- added TVS11: AIN1 low-leakage ESD, DIY_DASH:SOD323, symbol Connector_Generic:Conn_01x02
- added TVS12: AIN2 low-leakage ESD, DIY_DASH:SOD323, symbol Connector_Generic:Conn_01x02
- added TVS13: AIN3 low-leakage ESD, DIY_DASH:SOD323, symbol Connector_Generic:Conn_01x02
- added TVS14: AIN4 low-leakage ESD, DIY_DASH:SOD323, symbol Connector_Generic:Conn_01x02
- added TVS15: AIN5 low-leakage ESD, DIY_DASH:SOD323, symbol Connector_Generic:Conn_01x02
- added TVS16: AIN6 low-leakage ESD, DIY_DASH:SOD323, symbol Connector_Generic:Conn_01x02
- added TVS17: AIN7 low-leakage ESD, DIY_DASH:SOD323, symbol Connector_Generic:Conn_01x02
- added TVS18: AIN8 low-leakage ESD, DIY_DASH:SOD323, symbol Connector_Generic:Conn_01x02
- added U1: STM32G0B1CBT6, DIY_DASH:LQFP-48_7x7mm, symbol Connector_Generic:Conn_01x48
- added U10: MAX31855KASA+, DIY_DASH:SOIC-8_narrow, symbol Connector_Generic:Conn_01x08
- added U11: Schmitt Flex front end, DIY_DASH:SOT-353, symbol Connector_Generic:Conn_01x05
- added U2: LMR16006Y-Q1, DIY_DASH:SOT-23-THN-6_DDC, symbol Connector_Generic:Conn_01x06
- added U3: 3V3 LDO 300mA, DIY_DASH:SOT-23-5, symbol Connector_Generic:Conn_01x05
- added U4: SENSOR_5V load switch, DIY_DASH:SC70-5, symbol Connector_Generic:Conn_01x05
- added U5: 74HCT4051 1K excitation, DIY_DASH:SOIC-16, symbol Connector_Generic:Conn_01x16
- added U6: 74HCT4051 4K7 excitation, DIY_DASH:SOIC-16, symbol Connector_Generic:Conn_01x16
- added U7: L9613, DIY_DASH:SO-8, symbol Connector_Generic:Conn_01x08
- added U8: TJA1051T/3, DIY_DASH:SO-8_SOT96-1, symbol Connector_Generic:Conn_01x08
- added U9: TLV9002-Q1, DIY_DASH:SOIC-8, symbol Connector_Generic:Conn_01x08
Connections:
- new net +3V3: C3.1 (Pin_1), C4.1 (Pin_1), C5.1 (Pin_1), FB1.1 (Pin_1), J2.1 (Pin_1), R9.1 (Pin_1), U1.4 (Pin_4), U1.6 (Pin_6), U10.4 (Pin_4), U11.5 (Pin_5), U3.5 (Pin_5), U8.5 (Pin_5)
- new net +5V: C2.1 (Pin_1), L1.2 (Pin_2), R1.1 (Pin_1), R2.1 (Pin_1), R3.1 (Pin_1), R4.1 (Pin_1), U3.1 (Pin_1), U3.3 (Pin_3), U4.5 (Pin_5), U5.16 (Pin_16), U6.16 (Pin_16), U7.3 (Pin_3), U8.3 (Pin_3), U9.8 (Pin_8)
- new net ADC_IN1: C101.1 (Pin_1), R101.2 (Pin_2), R111.1 (Pin_1), U1.11 (Pin_11)
- new net ADC_IN2: C102.1 (Pin_1), R102.2 (Pin_2), R112.1 (Pin_1), U1.12 (Pin_12)
- new net ADC_IN3: C103.1 (Pin_1), R103.2 (Pin_2), R113.1 (Pin_1), U1.13 (Pin_13)
- new net ADC_IN4: C104.1 (Pin_1), R104.2 (Pin_2), R114.1 (Pin_1), U1.14 (Pin_14)
- new net ADC_IN5: C105.1 (Pin_1), R105.2 (Pin_2), R115.1 (Pin_1), U1.17 (Pin_17)
- new net ADC_IN6: C106.1 (Pin_1), R106.2 (Pin_2), R116.1 (Pin_1), U1.18 (Pin_18)
- new net ADC_IN7: C107.1 (Pin_1), R107.2 (Pin_2), R117.1 (Pin_1), U1.19 (Pin_19)
- new net ADC_IN8: C108.1 (Pin_1), R108.2 (Pin_2), R118.1 (Pin_1), U1.20 (Pin_20)
- new net AIN1: J1.9 (Pin_9), R101.1 (Pin_1), TVS11.1 (Pin_1), U5.13 (Pin_13), U6.13 (Pin_13)
- new net AIN2: J1.10 (Pin_10), R102.1 (Pin_1), TVS12.1 (Pin_1), U5.14 (Pin_14), U6.14 (Pin_14)
- new net AIN3: J1.11 (Pin_11), R103.1 (Pin_1), TVS13.1 (Pin_1), U5.15 (Pin_15), U6.15 (Pin_15)
- new net AIN4: J1.12 (Pin_12), R104.1 (Pin_1), TVS14.1 (Pin_1), U5.12 (Pin_12), U6.12 (Pin_12)
- new net AIN5: J1.13 (Pin_13), R105.1 (Pin_1), TVS15.1 (Pin_1), U5.1 (Pin_1), U6.1 (Pin_1)
- new net AIN6: J1.14 (Pin_14), R106.1 (Pin_1), TVS16.1 (Pin_1), U5.5 (Pin_5), U6.5 (Pin_5)
- new net AIN7: J1.15 (Pin_15), R107.1 (Pin_1), TVS17.1 (Pin_1), U5.2 (Pin_2), U6.2 (Pin_2)
- new net AIN8: J1.16 (Pin_16), R108.1 (Pin_1), TVS18.1 (Pin_1), U5.4 (Pin_4), U6.4 (Pin_4)
- new net AOUT1: D6.1 (Pin_1), J1.22 (Pin_22), R7.2 (Pin_2)
- new net AOUT1_OP: R7.1 (Pin_1), U9.2 (Pin_2), U9.3 (Pin_3)
- new net AOUT2: D7.1 (Pin_1), J1.23 (Pin_23), R8.2 (Pin_2)
- new net AOUT2_OP: R8.1 (Pin_1), U9.6 (Pin_6), U9.7 (Pin_7)
- new net BOOT0: R10.1 (Pin_1), U1.21 (Pin_21)
- new net BUCK_BOOT: U2.1 (Pin_1)
- new net BUCK_FB: U2.3 (Pin_3)
- new net BUCK_SW: D2.2 (Pin_2), L1.1 (Pin_1), U2.6 (Pin_6)
- new net CAN_H: D3.1 (Pin_1), J1.4 (Pin_4), JP1.1 (Pin_1), L2.3 (Pin_3)
- new net CAN_H_PROTECTED: L2.1 (Pin_1), U8.7 (Pin_7)
- new net CAN_L: D3.2 (Pin_2), J1.5 (Pin_5), JP1.2 (Pin_2), L2.4 (Pin_4)
- new net CAN_L_PROTECTED: L2.2 (Pin_2), U8.6 (Pin_6)
- new net CAN_RX: U1.33 (Pin_33), U8.4 (Pin_4)
- new net CAN_SILENT: U1.26 (Pin_26), U8.8 (Pin_8)
- new net CAN_TX: U1.34 (Pin_34), U8.1 (Pin_1)
- new net DAC1_RAW: U1.15 (Pin_15), U9.1 (Pin_1)
- new net DAC2_RAW: U1.16 (Pin_16), U9.5 (Pin_5)
- new net EGT_CS: U1.44 (Pin_44), U10.6 (Pin_6)
- new net EGT_K_NEG: J1.18 (Pin_18), U10.3 (Pin_3)
- new net EGT_K_POS: J1.17 (Pin_17), U10.2 (Pin_2)
- new net EGT_SCK: U1.42 (Pin_42), U10.5 (Pin_5)
- new net EGT_SO: U1.43 (Pin_43), U10.7 (Pin_7)
- new net EXC_1K: R1.2 (Pin_2), U5.3 (Pin_3)
- new net EXC_4K7: R2.2 (Pin_2), U6.3 (Pin_3)
- new net FLEX_CAPTURE: U1.28 (Pin_28), U11.4 (Pin_4)
- new net FLEX_IN: D5.1 (Pin_1), J1.21 (Pin_21), U11.2 (Pin_2)
- new net IGN: J1.3 (Pin_3), Q1.1 (Pin_1), U2.4 (Pin_4)
- new net IGN_SENSE: U1.29 (Pin_29)
- new net KLINE_ENABLE: U1.37 (Pin_37)
- new net KRX: U1.46 (Pin_46), U7.1 (Pin_1)
- new net KTX: U1.45 (Pin_45), U7.4 (Pin_4)
- new net K_LINE: D4.1 (Pin_1), J1.6 (Pin_6), U7.6 (Pin_6)
- new net NRST: J2.4 (Pin_4), R9.2 (Pin_2), TP3.1 (Pin_1), U1.10 (Pin_10)
- new net POWER_GND: C1.2 (Pin_2), C2.2 (Pin_2), C3.2 (Pin_2), C4.2 (Pin_2), C5.2 (Pin_2), C6.2 (Pin_2), D1.2 (Pin_2), D2.1 (Pin_1), D4.2 (Pin_2), D5.2 (Pin_2), D6.2 (Pin_2), D7.2 (Pin_2), J1.2 (Pin_2), J2.5 (Pin_5), Q4.3 (Pin_3), Q5.3 (Pin_3), R10.2 (Pin_2), R5.2 (Pin_2), R6.2 (Pin_2), TVS11.2 (Pin_2), TVS12.2 (Pin_2), TVS13.2 (Pin_2), TVS14.2 (Pin_2), TVS15.2 (Pin_2), TVS16.2 (Pin_2), TVS17.2 (Pin_2), TVS18.2 (Pin_2), U1.7 (Pin_7), U10.1 (Pin_1), U11.3 (Pin_3), U2.2 (Pin_2), U3.2 (Pin_2), U4.2 (Pin_2), U5.7 (Pin_7), U5.8 (Pin_8), U6.7 (Pin_7), U6.8 (Pin_8), U7.5 (Pin_5), U8.2 (Pin_2), U9.4 (Pin_4)
- new net PULL_1K_EN_N: R3.2 (Pin_2), U1.41 (Pin_41), U5.6 (Pin_6)
- new net PULL_4K7_EN_N: R4.2 (Pin_2), U1.30 (Pin_30), U6.6 (Pin_6)
- new net PULL_A0: U1.38 (Pin_38), U5.11 (Pin_11), U6.11 (Pin_11)
- new net PULL_A1: U1.39 (Pin_39), U5.10 (Pin_10), U6.10 (Pin_10)
- new net PULL_A2: U1.40 (Pin_40), U5.9 (Pin_9), U6.9 (Pin_9)
- new net RELAY1_GATE: Q4.1 (Pin_1), R5.1 (Pin_1), U1.31 (Pin_31)
- new net RELAY2_GATE: Q5.1 (Pin_1), R6.1 (Pin_1), U1.25 (Pin_25)
- new net RELAY_OUT1: J1.19 (Pin_19), Q4.2 (Pin_2), Q4.4 (Pin_4), Q4.5 (Pin_5), Q4.6 (Pin_6), Q4.7 (Pin_7), Q4.8 (Pin_8)
- new net RELAY_OUT2: J1.20 (Pin_20), Q5.2 (Pin_2), Q5.4 (Pin_4), Q5.5 (Pin_5), Q5.6 (Pin_6), Q5.7 (Pin_7), Q5.8 (Pin_8)
- new net SENSOR_5V: F2.2 (Pin_2), J1.7 (Pin_7)
- new net SENSOR_5V_EN: U1.27 (Pin_27), U4.4 (Pin_4)
- new net SENSOR_5V_OC: U4.3 (Pin_3)
- new net SENSOR_5V_SW: F2.1 (Pin_1), U4.1 (Pin_1)
- new net SENSOR_GND: C101.2 (Pin_2), C102.2 (Pin_2), C103.2 (Pin_2), C104.2 (Pin_2), C105.2 (Pin_2), C106.2 (Pin_2), C107.2 (Pin_2), C108.2 (Pin_2), J1.8 (Pin_8), R111.2 (Pin_2), R112.2 (Pin_2), R113.2 (Pin_2), R114.2 (Pin_2), R115.2 (Pin_2), R116.2 (Pin_2), R117.2 (Pin_2), R118.2 (Pin_2)
- new net SERVICE: J1.24 (Pin_24), U1.32 (Pin_32)
- new net SWCLK: J2.3 (Pin_3), TP2.1 (Pin_1), U1.36 (Pin_36)
- new net SWDIO: J2.2 (Pin_2), TP1.1 (Pin_1), U1.35 (Pin_35)
- new net V3V3_MON: U1.24 (Pin_24)
- new net V5_MON: U1.23 (Pin_23)
- new net VBAT: F1.1 (Pin_1), J1.1 (Pin_1)
- new net VBAT_FUSED: F1.2 (Pin_2), Q1.3 (Pin_3), Q1.4 (Pin_4)
- new net VBAT_MON: U1.22 (Pin_22)
- new net VBAT_PROTECTED: C1.1 (Pin_1), D1.1 (Pin_1), Q1.2 (Pin_2), U2.5 (Pin_5), U7.7 (Pin_7)
- new net VDDA: C6.1 (Pin_1), FB1.2 (Pin_2), U1.5 (Pin_5)
- no-connect marks 0 -> 12
Other:
- note added: "C1 / 1210"
- note added: "C101 / 0603"
- note added: "C102 / 0603"
- note added: "C103 / 0603"
- note added: "C104 / 0603"
- note added: "C105 / 0603"
- note added: "C106 / 0603"
- note added: "C107 / 0603"
- note added: "C108 / 0603"
- note added: "C2 / 1206"
- note added: "C3 / 0805"
- note added: "C4 / 0603"
- note added: "C5 / 0603"
- note added: "C6 / 0603"
- note added: "CAN I/O MODULE - ELECTRICAL SOURCE OF TRUTH"
- note added: "D1 / SMB DO-214AA"
- note added: "D2 / SMA DO-214AC"
- note added: "D3 / SOT23"
- note added: "D4 / SMA DO-214AC"
- note added: "D5 / SOD323"
- note added: "D6 / SOD323"
- note added: "D7 / SOD323"
- note added: "Every net label is wired to the numbered physical package pin. J2: 1 +3V3, 2 SWDIO, 3 SWCLK, 4 NRST, 5 POWER_GND."
- note added: "F1 / NANO2 2410"
- note added: "F2 / 1206"
- note added: "FB1 / 0603"
- note added: "J1 / Custom THT 3x8"
- note added: "J2 / PinHeader_1x05_P2.54mm_Vertical"
- note added: "JP1 / 0603"
- note added: "L1 / 5.5x5.5mm"
- note added: "L2 / 1812 common-mode"
- note added: "Q1 / PowerPAK SO-8"
- note added: "Q4 / LFPAK56"
- note added: "Q5 / LFPAK56"
- note added: "R1 / 0603"
- note added: "R10 / 0603"
- note added: "R101 / 0603"
- note added: "R102 / 0603"
- note added: "R103 / 0603"
- note added: "R104 / 0603"
- note added: "R105 / 0603"
- note added: "R106 / 0603"
- note added: "R107 / 0603"
- note added: "R108 / 0603"
- note added: "R111 / 0603"
- note added: "R112 / 0603"
- note added: "R113 / 0603"
- note added: "R114 / 0603"
- note added: "R115 / 0603"
- note added: "R116 / 0603"
- note added: "R117 / 0603"
- note added: "R118 / 0603"
- note added: "R2 / 0603"
- note added: "R3 / 0603"
- note added: "R4 / 0603"
- note added: "R5 / 0603"
- note added: "R6 / 0603"
- note added: "R7 / 0603"
- note added: "R8 / 0603"
- note added: "R9 / 0603"
- note added: "TP1 / Test pad"
- note added: "TP2 / Test pad"
- note added: "TP3 / Test pad"
- note added: "TVS11 / SOD323"
- note added: "TVS12 / SOD323"
- note added: "TVS13 / SOD323"
- note added: "TVS14 / SOD323"
- note added: "TVS15 / SOD323"
- note added: "TVS16 / SOD323"
- note added: "TVS17 / SOD323"
- note added: "TVS18 / SOD323"
- note added: "U1 / LQFP-48 7x7mm"
- note added: "U10 / SOIC-8 narrow"
- note added: "U11 / SOT-353"
- note added: "U2 / SOT-23-THN-6 DDC"
- note added: "U3 / SOT-23-5"
- note added: "U4 / SC70-5"
- note added: "U5 / SOIC-16"
- note added: "U6 / SOIC-16"
- note added: "U7 / SO-8"
- note added: "U8 / SO-8 SOT96-1"
- note added: "U9 / SOIC-8"
- note removed: "CAN I/O MODULE - HIERARCHICAL INDEX"
- note removed: "J1 ECU_FCI_24P: fixed pinout 1..24 defined in project README"
- note removed: "PROTOTYPE ONLY - verify connector and enclosure before fabrication"
- note removed: "SHEET 2 power.kicad_sch: protected VBAT, 5V, 3V3, IGN and rail monitors"
- note removed: "SHEET 3 mcu.kicad_sch: STM32G0B1CBT6, SWD, reset, ADC/DAC/timers"
- note removed: "SHEET 4 analog-inputs.kicad_sch: eight identical protected universal inputs"
- note removed: "SHEET 5 communications-egt.kicad_sch: CAN, L9613 K-line, EGT and Flex Fuel"
- note removed: "SHEET 6 outputs.kicad_sch: two 0-5V signals and two low-side relay drivers"
- title: CAN I/O MODULE - HIERARCHICAL INDEX -> DIY Dash 5 CAN I/O Module

Commit message: fix: render explicit CAN IO schematic wiring
Connections:
- net +3V3: now also J2.5 (Pin_5), U1.42 (Pin_42), U1.44 (Pin_44), U11.1 (Pin_1), U3.1 (Pin_1), U8.3 (Pin_3); no longer J2.1 (Pin_1), U1.4 (Pin_4), U1.6 (Pin_6), U11.5 (Pin_5), U3.5 (Pin_5), U8.5 (Pin_5)
- net +5V: now also U3.5 (Pin_5), U4.1 (Pin_1), U7.5 (Pin_5), U8.5 (Pin_5); no longer L1.2 (Pin_2), U3.1 (Pin_1), U4.5 (Pin_5), U5.16 (Pin_16), U6.16 (Pin_16), U7.3 (Pin_3), U8.3 (Pin_3), U9.8 (Pin_8)
- net ADC_IN1: now also U1.37 (Pin_37); no longer R101.2 (Pin_2), U1.11 (Pin_11)
- net ADC_IN2: now also U1.36 (Pin_36); no longer R102.2 (Pin_2), U1.12 (Pin_12)
- net ADC_IN3: now also U1.35 (Pin_35); no longer R103.2 (Pin_2), U1.13 (Pin_13)
- net ADC_IN4: now also U1.34 (Pin_34); no longer R104.2 (Pin_2), U1.14 (Pin_14)
- net ADC_IN5: now also U1.31 (Pin_31); no longer R105.2 (Pin_2), U1.17 (Pin_17)
- net ADC_IN6: now also U1.30 (Pin_30); no longer R106.2 (Pin_2), U1.18 (Pin_18)
- net ADC_IN7: now also U1.29 (Pin_29); no longer R107.2 (Pin_2), U1.19 (Pin_19)
- net ADC_IN8: now also U1.28 (Pin_28); no longer R108.2 (Pin_2), U1.20 (Pin_20)
- net AIN1: now also J1.15 (Pin_15), U5.3 (Pin_3), U6.3 (Pin_3); no longer J1.9 (Pin_9), U5.13 (Pin_13), U6.13 (Pin_13)
- net AIN2: now also J1.14 (Pin_14), U5.2 (Pin_2), U6.2 (Pin_2); no longer J1.10 (Pin_10), U5.14 (Pin_14), U6.14 (Pin_14)
- net AIN3: now also J1.13 (Pin_13), U5.1 (Pin_1), U6.1 (Pin_1); no longer J1.11 (Pin_11), U5.15 (Pin_15), U6.15 (Pin_15)
- net AIN4: now also U5.4 (Pin_4), U6.4 (Pin_4); no longer U5.12 (Pin_12), U6.12 (Pin_12)
- net AIN5: now also J1.11 (Pin_11), U5.15 (Pin_15), U6.15 (Pin_15); no longer J1.13 (Pin_13), U5.1 (Pin_1), U6.1 (Pin_1)
- net AIN6: now also J1.10 (Pin_10), U5.11 (Pin_11), U6.11 (Pin_11); no longer J1.14 (Pin_14), U5.5 (Pin_5), U6.5 (Pin_5)
- net AIN7: now also J1.9 (Pin_9), U5.14 (Pin_14), U6.14 (Pin_14); no longer J1.15 (Pin_15), U5.2 (Pin_2), U6.2 (Pin_2)
- net AIN8: now also J1.8 (Pin_8), U5.12 (Pin_12), U6.12 (Pin_12); no longer J1.16 (Pin_16), U5.4 (Pin_4), U6.4 (Pin_4)
- net AOUT1: now also J1.2 (Pin_2); no longer J1.22 (Pin_22), R7.2 (Pin_2)
- net AOUT1_OP: now also U9.5 (Pin_5), U9.6 (Pin_6); no longer U9.2 (Pin_2), U9.3 (Pin_3)
- net AOUT2: now also J1.1 (Pin_1); no longer J1.23 (Pin_23), R8.2 (Pin_2)
- net AOUT2_OP: now also U9.1 (Pin_1), U9.2 (Pin_2); no longer U9.6 (Pin_6), U9.7 (Pin_7)
- net BOOT0: now also U1.27 (Pin_27); no longer U1.21 (Pin_21)
- net BUCK_BOOT: now also U2.5 (Pin_5); no longer U2.1 (Pin_1)
- net BUCK_SW: no longer D2.2 (Pin_2), U2.6 (Pin_6)
- net CAN_H: now also J1.20 (Pin_20), L2.1 (Pin_1); no longer J1.4 (Pin_4), L2.3 (Pin_3)
- net CAN_H_PROTECTED: now also L2.3 (Pin_3), U8.1 (Pin_1); no longer L2.1 (Pin_1), U8.7 (Pin_7)
- net CAN_L: now also J1.19 (Pin_19); no longer D3.2 (Pin_2), J1.5 (Pin_5), JP1.2 (Pin_2), L2.4 (Pin_4)
- net CAN_L_PROTECTED: now also U8.2 (Pin_2); no longer U8.6 (Pin_6)
- net CAN_RX: now also U1.15 (Pin_15); no longer U1.33 (Pin_33)
- net CAN_SILENT: now also U1.22 (Pin_22); no longer U1.26 (Pin_26), U8.8 (Pin_8)
- net CAN_TX: now also U1.14 (Pin_14), U8.7 (Pin_7); no longer U1.34 (Pin_34), U8.1 (Pin_1)
- net DAC1_RAW: now also U1.33 (Pin_33), U9.7 (Pin_7); no longer U1.15 (Pin_15), U9.1 (Pin_1)
- net DAC2_RAW: now also U1.32 (Pin_32), U9.3 (Pin_3); no longer U1.16 (Pin_16), U9.5 (Pin_5)
- net EGT_CS: now also U1.4 (Pin_4), U10.2 (Pin_2); no longer U1.44 (Pin_44), U10.6 (Pin_6)
- net EGT_K_NEG: now also J1.6 (Pin_6), U10.5 (Pin_5); no longer J1.18 (Pin_18), U10.3 (Pin_3)
- net EGT_K_POS: now also J1.7 (Pin_7), U10.6 (Pin_6); no longer J1.17 (Pin_17), U10.2 (Pin_2)
- net EGT_SCK: now also U1.6 (Pin_6), U10.3 (Pin_3); no longer U1.42 (Pin_42), U10.5 (Pin_5)
- net EGT_SO: now also U1.5 (Pin_5), U10.1 (Pin_1); no longer U1.43 (Pin_43), U10.7 (Pin_7)
- net EXC_1K: now also U5.13 (Pin_13); no longer R1.2 (Pin_2), U5.3 (Pin_3)
- net EXC_4K7: now also U6.13 (Pin_13); no longer R2.2 (Pin_2), U6.3 (Pin_3)
- net FLEX_CAPTURE: now also U1.20 (Pin_20), U11.2 (Pin_2); no longer U1.28 (Pin_28), U11.4 (Pin_4)
- net FLEX_IN: now also J1.3 (Pin_3), U11.4 (Pin_4); no longer J1.21 (Pin_21), U11.2 (Pin_2)
- net IGN: now also J1.21 (Pin_21), Q1.3 (Pin_3), U2.2 (Pin_2); no longer J1.3 (Pin_3), Q1.1 (Pin_1), U2.4 (Pin_4)
- net IGN_SENSE: now also U1.19 (Pin_19); no longer U1.29 (Pin_29)
- net KLINE_ENABLE: now also U1.11 (Pin_11); no longer U1.37 (Pin_37)
- net KRX: now also U1.2 (Pin_2), U7.7 (Pin_7); no longer U1.46 (Pin_46), U7.1 (Pin_1)
- net KTX: now also U1.3 (Pin_3); no longer U1.45 (Pin_45)
- net K_LINE: now also J1.18 (Pin_18), U7.2 (Pin_2); no longer J1.6 (Pin_6), U7.6 (Pin_6)
- net NRST: now also J2.2 (Pin_2), U1.38 (Pin_38); no longer J2.4 (Pin_4), R9.2 (Pin_2), U1.10 (Pin_10)
- net POWER_GND: now also J1.22 (Pin_22), J2.1 (Pin_1), Q4.5 (Pin_5), Q5.5 (Pin_5), U1.41 (Pin_41), U10.7 (Pin_7), U2.4 (Pin_4), U3.4 (Pin_4), U4.4 (Pin_4), U5.9 (Pin_9), U6.9 (Pin_9), U7.3 (Pin_3), U8.6 (Pin_6); no longer C1.2 (Pin_2), C2.2 (Pin_2), C3.2 (Pin_2), C4.2 (Pin_2), C5.2 (Pin_2), C6.2 (Pin_2), D1.2 (Pin_2), D4.2 (Pin_2), D5.2 (Pin_2), D6.2 (Pin_2), D7.2 (Pin_2), J1.2 (Pin_2), J2.5 (Pin_5), Q4.3 (Pin_3), Q5.3 (Pin_3), R10.2 (Pin_2), R5.2 (Pin_2), R6.2 (Pin_2), TVS11.2 (Pin_2), TVS12.2 (Pin_2), TVS13.2 (Pin_2), TVS14.2 (Pin_2), TVS15.2 (Pin_2), TVS16.2 (Pin_2), TVS17.2 (Pin_2), TVS18.2 (Pin_2), U1.7 (Pin_7), U10.1 (Pin_1), U2.2 (Pin_2), U3.2 (Pin_2), U4.2 (Pin_2), U5.7 (Pin_7), U6.7 (Pin_7), U7.5 (Pin_5), U8.2 (Pin_2)
- net PULL_1K_EN_N: now also U1.7 (Pin_7), U5.10 (Pin_10); no longer R3.2 (Pin_2), U1.41 (Pin_41), U5.6 (Pin_6)
- net PULL_4K7_EN_N: now also U1.18 (Pin_18), U6.10 (Pin_10); no longer R4.2 (Pin_2), U1.30 (Pin_30), U6.6 (Pin_6)
- net PULL_A0: now also U1.10 (Pin_10), U5.5 (Pin_5), U6.5 (Pin_5); no longer U1.38 (Pin_38), U5.11 (Pin_11), U6.11 (Pin_11)
- net PULL_A1: now also U1.9 (Pin_9), U5.6 (Pin_6), U6.6 (Pin_6); no longer U1.39 (Pin_39), U5.10 (Pin_10), U6.10 (Pin_10)
- net PULL_A2: now also U1.8 (Pin_8), U5.7 (Pin_7), U6.7 (Pin_7); no longer U1.40 (Pin_40), U5.9 (Pin_9), U6.9 (Pin_9)
- net RELAY1_GATE: now also Q4.7 (Pin_7), U1.17 (Pin_17); no longer Q4.1 (Pin_1), U1.31 (Pin_31)
- net RELAY2_GATE: now also Q5.7 (Pin_7), U1.23 (Pin_23); no longer Q5.1 (Pin_1), U1.25 (Pin_25)
- net RELAY_OUT1: now also J1.5 (Pin_5), Q4.1 (Pin_1), Q4.3 (Pin_3); no longer J1.19 (Pin_19), Q4.5 (Pin_5), Q4.7 (Pin_7), Q4.8 (Pin_8)
- net RELAY_OUT2: now also J1.4 (Pin_4), Q5.1 (Pin_1), Q5.3 (Pin_3); no longer J1.20 (Pin_20), Q5.5 (Pin_5), Q5.7 (Pin_7), Q5.8 (Pin_8)
- net SENSOR_5V: now also J1.17 (Pin_17); no longer F2.2 (Pin_2), J1.7 (Pin_7)
- net SENSOR_5V_EN: now also U1.21 (Pin_21), U4.2 (Pin_2); no longer U1.27 (Pin_27), U4.4 (Pin_4)
- net SENSOR_5V_SW: now also U4.5 (Pin_5); no longer U4.1 (Pin_1)
- net SENSOR_GND: now also J1.16 (Pin_16); no longer C101.2 (Pin_2), C102.2 (Pin_2), C103.2 (Pin_2), C104.2 (Pin_2), C105.2 (Pin_2), C106.2 (Pin_2), C107.2 (Pin_2), C108.2 (Pin_2), J1.8 (Pin_8), R111.2 (Pin_2), R112.2 (Pin_2), R113.2 (Pin_2), R114.2 (Pin_2), R115.2 (Pin_2), R116.2 (Pin_2), R117.2 (Pin_2), R118.2 (Pin_2)
- net SERVICE: now also U1.16 (Pin_16); no longer J1.24 (Pin_24), U1.32 (Pin_32)
- net SWCLK: now also U1.12 (Pin_12); no longer U1.36 (Pin_36)
- net SWDIO: now also J2.4 (Pin_4), U1.13 (Pin_13); no longer J2.2 (Pin_2), U1.35 (Pin_35)
- net V5_MON: now also U1.25 (Pin_25); no longer U1.23 (Pin_23)
- net VBAT: now also J1.23 (Pin_23); no longer J1.1 (Pin_1)
- net VBAT_FUSED: now also Q1.1 (Pin_1); no longer F1.2 (Pin_2), Q1.3 (Pin_3), Q1.4 (Pin_4)
- net VBAT_MON: now also U1.26 (Pin_26); no longer U1.22 (Pin_22)
- net VBAT_PROTECTED: now also U2.1 (Pin_1), U7.1 (Pin_1); no longer U2.5 (Pin_5), U7.7 (Pin_7)
- net VDDA: now also U1.43 (Pin_43); no longer FB1.2 (Pin_2), U1.5 (Pin_5)

Commit message: fix: make CAN IO symbol and footprint libraries self contained
Parts:
- J2: footprint Connector_PinHeader_2.54mm:PinHeader_1x05_P2.54mm_Vertical -> DIY_DASH:SWD_1x05_P2.54mm_Vertical

Commit message: fix: use explicit global net endpoints in CAN IO schematic
Connections:
- removed net +3V3: C3.1 (Pin_1), C4.1 (Pin_1), C5.1 (Pin_1), FB1.1 (Pin_1), J2.5 (Pin_5), R9.1 (Pin_1), U1.42 (Pin_42), U1.44 (Pin_44), U10.4 (Pin_4), U11.1 (Pin_1), U3.1 (Pin_1), U8.3 (Pin_3)
- removed net +5V: C2.1 (Pin_1), R1.1 (Pin_1), R2.1 (Pin_1), R3.1 (Pin_1), R4.1 (Pin_1), U3.3 (Pin_3), U3.5 (Pin_5), U4.1 (Pin_1), U7.5 (Pin_5), U8.5 (Pin_5)
- removed net ADC_IN1: C101.1 (Pin_1), R111.1 (Pin_1), U1.37 (Pin_37)
- removed net ADC_IN2: C102.1 (Pin_1), R112.1 (Pin_1), U1.36 (Pin_36)
- removed net ADC_IN3: C103.1 (Pin_1), R113.1 (Pin_1), U1.35 (Pin_35)
- removed net ADC_IN4: C104.1 (Pin_1), R114.1 (Pin_1), U1.34 (Pin_34)
- removed net ADC_IN5: C105.1 (Pin_1), R115.1 (Pin_1), U1.31 (Pin_31)
- removed net ADC_IN6: C106.1 (Pin_1), R116.1 (Pin_1), U1.30 (Pin_30)
- removed net ADC_IN7: C107.1 (Pin_1), R117.1 (Pin_1), U1.29 (Pin_29)
- removed net ADC_IN8: C108.1 (Pin_1), R118.1 (Pin_1), U1.28 (Pin_28)
- removed net AIN1: J1.15 (Pin_15), R101.1 (Pin_1), TVS11.1 (Pin_1), U5.3 (Pin_3), U6.3 (Pin_3)
- removed net AIN2: J1.14 (Pin_14), R102.1 (Pin_1), TVS12.1 (Pin_1), U5.2 (Pin_2), U6.2 (Pin_2)
- removed net AIN3: J1.13 (Pin_13), R103.1 (Pin_1), TVS13.1 (Pin_1), U5.1 (Pin_1), U6.1 (Pin_1)
- removed net AIN4: J1.12 (Pin_12), R104.1 (Pin_1), TVS14.1 (Pin_1), U5.4 (Pin_4), U6.4 (Pin_4)
- removed net AIN5: J1.11 (Pin_11), R105.1 (Pin_1), TVS15.1 (Pin_1), U5.15 (Pin_15), U6.15 (Pin_15)
- removed net AIN6: J1.10 (Pin_10), R106.1 (Pin_1), TVS16.1 (Pin_1), U5.11 (Pin_11), U6.11 (Pin_11)
- removed net AIN7: J1.9 (Pin_9), R107.1 (Pin_1), TVS17.1 (Pin_1), U5.14 (Pin_14), U6.14 (Pin_14)
- removed net AIN8: J1.8 (Pin_8), R108.1 (Pin_1), TVS18.1 (Pin_1), U5.12 (Pin_12), U6.12 (Pin_12)
- net AOUT1: no longer names the net of J1.2 (Pin_2)
- net AOUT1: no longer D6.1 (Pin_1)
- removed net AOUT1_OP: R7.1 (Pin_1), U9.5 (Pin_5), U9.6 (Pin_6)
- net AOUT2: no longer names the net of J1.1 (Pin_1)
- net AOUT2: no longer D7.1 (Pin_1)
- removed net AOUT2_OP: R8.1 (Pin_1), U9.1 (Pin_1), U9.2 (Pin_2)
- net BOOT0: no longer names the net of U1.27 (Pin_27)
- net BOOT0: no longer R10.1 (Pin_1)
- net BUCK_BOOT: no longer names the net of U2.5 (Pin_5)
- net BUCK_FB: no longer names the net of U2.3 (Pin_3)
- net BUCK_SW: no longer names the net of L1.1 (Pin_1)
- removed net CAN_H: D3.1 (Pin_1), J1.20 (Pin_20), JP1.1 (Pin_1), L2.1 (Pin_1)
- net CAN_H_PROTECTED: no longer names the net of L2.3 (Pin_3)
- net CAN_H_PROTECTED: no longer U8.1 (Pin_1)
- net CAN_L: no longer names the net of J1.19 (Pin_19)
- net CAN_L_PROTECTED: no longer names the net of L2.2 (Pin_2)
- net CAN_L_PROTECTED: no longer U8.2 (Pin_2)
- net CAN_RX: no longer names the net of U8.4 (Pin_4)
- net CAN_RX: no longer U1.15 (Pin_15)
- net CAN_SILENT: no longer names the net of U1.22 (Pin_22)
- net CAN_TX: no longer names the net of U8.7 (Pin_7)
- net CAN_TX: no longer U1.14 (Pin_14)
- net DAC1_RAW: no longer names the net of U1.33 (Pin_33)
- net DAC1_RAW: no longer U9.7 (Pin_7)
- net DAC2_RAW: no longer names the net of U1.32 (Pin_32)
- net DAC2_RAW: no longer U9.3 (Pin_3)
- net EGT_CS: no longer names the net of U1.4 (Pin_4)
- net EGT_CS: no longer U10.2 (Pin_2)
- net EGT_K_NEG: no longer names the net of J1.6 (Pin_6)
- net EGT_K_NEG: no longer U10.5 (Pin_5)
- net EGT_K_POS: no longer names the net of J1.7 (Pin_7)
- net EGT_K_POS: no longer U10.6 (Pin_6)
- net EGT_SCK: no longer names the net of U1.6 (Pin_6)
- net EGT_SCK: no longer U10.3 (Pin_3)
- net EGT_SO: no longer names the net of U1.5 (Pin_5)
- net EGT_SO: no longer U10.1 (Pin_1)
- net EXC_1K: no longer names the net of U5.13 (Pin_13)
- net EXC_4K7: no longer names the net of U6.13 (Pin_13)
- net FLEX_CAPTURE: no longer names the net of U11.2 (Pin_2)
- net FLEX_CAPTURE: no longer U1.20 (Pin_20)
- removed net FLEX_IN: D5.1 (Pin_1), J1.3 (Pin_3), U11.4 (Pin_4)
- removed net IGN: J1.21 (Pin_21), Q1.3 (Pin_3), U2.2 (Pin_2)
- net IGN_SENSE: no longer names the net of U1.19 (Pin_19)
- net KLINE_ENABLE: no longer names the net of U1.11 (Pin_11)
- net KRX: no longer names the net of U1.2 (Pin_2)
- net KRX: no longer U7.7 (Pin_7)
- net KTX: no longer names the net of U1.3 (Pin_3)
- net KTX: no longer U7.4 (Pin_4)
- removed net K_LINE: D4.1 (Pin_1), J1.18 (Pin_18), U7.2 (Pin_2)
- removed net NRST: J2.2 (Pin_2), TP3.1 (Pin_1), U1.38 (Pin_38)
- removed net POWER_GND: D2.1 (Pin_1), J1.22 (Pin_22), J2.1 (Pin_1), Q4.5 (Pin_5), Q5.5 (Pin_5), U1.41 (Pin_41), U10.7 (Pin_7), U11.3 (Pin_3), U2.4 (Pin_4), U3.4 (Pin_4), U4.4 (Pin_4), U5.8 (Pin_8), U5.9 (Pin_9), U6.8 (Pin_8), U6.9 (Pin_9), U7.3 (Pin_3), U8.6 (Pin_6), U9.4 (Pin_4)
- net PULL_1K_EN_N: no longer names the net of U1.7 (Pin_7)
- net PULL_1K_EN_N: no longer U5.10 (Pin_10)
- net PULL_4K7_EN_N: no longer names the net of U6.10 (Pin_10)
- net PULL_4K7_EN_N: no longer U1.18 (Pin_18)
- removed net PULL_A0: U1.10 (Pin_10), U5.5 (Pin_5), U6.5 (Pin_5)
- removed net PULL_A1: U1.9 (Pin_9), U5.6 (Pin_6), U6.6 (Pin_6)
- removed net PULL_A2: U1.8 (Pin_8), U5.7 (Pin_7), U6.7 (Pin_7)
- removed net RELAY1_GATE: Q4.7 (Pin_7), R5.1 (Pin_1), U1.17 (Pin_17)
- removed net RELAY2_GATE: Q5.7 (Pin_7), R6.1 (Pin_1), U1.23 (Pin_23)
- removed net RELAY_OUT1: J1.5 (Pin_5), Q4.1 (Pin_1), Q4.2 (Pin_2), Q4.3 (Pin_3), Q4.4 (Pin_4), Q4.6 (Pin_6)
- removed net RELAY_OUT2: J1.4 (Pin_4), Q5.1 (Pin_1), Q5.2 (Pin_2), Q5.3 (Pin_3), Q5.4 (Pin_4), Q5.6 (Pin_6)
- net SENSOR_5V: no longer names the net of J1.17 (Pin_17)
- net SENSOR_5V_EN: no longer names the net of U4.2 (Pin_2)
- net SENSOR_5V_EN: no longer U1.21 (Pin_21)
- net SENSOR_5V_OC: no longer names the net of U4.3 (Pin_3)
- net SENSOR_5V_SW: no longer names the net of U4.5 (Pin_5)
- net SENSOR_5V_SW: no longer F2.1 (Pin_1)
- net SENSOR_GND: no longer names the net of J1.16 (Pin_16)
- net SERVICE: no longer names the net of U1.16 (Pin_16)
- removed net SWCLK: J2.3 (Pin_3), TP2.1 (Pin_1), U1.12 (Pin_12)
- removed net SWDIO: J2.4 (Pin_4), TP1.1 (Pin_1), U1.13 (Pin_13)
- net V3V3_MON: no longer names the net of U1.24 (Pin_24)
- net V5_MON: no longer names the net of U1.25 (Pin_25)
- net VBAT: no longer names the net of J1.23 (Pin_23)
- net VBAT: no longer F1.1 (Pin_1)
- net VBAT_FUSED: no longer names the net of Q1.1 (Pin_1)
- net VBAT_MON: no longer names the net of U1.26 (Pin_26)
- removed net VBAT_PROTECTED: C1.1 (Pin_1), D1.1 (Pin_1), Q1.2 (Pin_2), U2.1 (Pin_1), U7.1 (Pin_1)
- net VDDA: no longer names the net of U1.43 (Pin_43)
- net VDDA: no longer C6.1 (Pin_1)

Commit message: fix: connect equal CAN IO nets with physical wires
Connections:
- net +3V3: now reaches U11.2 (Pin_2)
- net +3V3: now also C1.1 (Pin_1), C1.2 (Pin_2), C101.1 (Pin_1), C101.2 (Pin_2), C102.1 (Pin_1), C102.2 (Pin_2), C103.1 (Pin_1), C103.2 (Pin_2), C104.1 (Pin_1), C104.2 (Pin_2), C105.1 (Pin_1), C105.2 (Pin_2), C106.1 (Pin_1), C106.2 (Pin_2), C107.1 (Pin_1), C107.2 (Pin_2), C108.1 (Pin_1), C108.2 (Pin_2), C2.1 (Pin_1), C2.2 (Pin_2), C3.1 (Pin_1), C3.2 (Pin_2), C4.1 (Pin_1), C4.2 (Pin_2), C5.1 (Pin_1), C5.2 (Pin_2), C6.1 (Pin_1), C6.2 (Pin_2), D1.1 (Pin_1), D1.2 (Pin_2), D2.1 (Pin_1), D2.2 (Pin_2), D3.1 (Pin_1), D3.2 (Pin_2), D4.1 (Pin_1), D4.2 (Pin_2), D5.1 (Pin_1), D5.2 (Pin_2), D6.1 (Pin_1), D6.2 (Pin_2), D7.1 (Pin_1), D7.2 (Pin_2), F1.1 (Pin_1), F1.2 (Pin_2), F2.1 (Pin_1), F2.2 (Pin_2), FB1.1 (Pin_1), FB1.2 (Pin_2), J1.1 (Pin_1), J1.10 (Pin_10), J1.11 (Pin_11), J1.12 (Pin_12), J1.13 (Pin_13), J1.14 (Pin_14), J1.16 (Pin_16), J1.17 (Pin_17), J1.18 (Pin_18), J1.19 (Pin_19), J1.2 (Pin_2), J1.20 (Pin_20), J1.21 (Pin_21), J1.22 (Pin_22), J1.23 (Pin_23), J1.24 (Pin_24), J1.3 (Pin_3), J1.4 (Pin_4), J1.5 (Pin_5), J1.6 (Pin_6), J1.7 (Pin_7), J1.8 (Pin_8), J1.9 (Pin_9), J2.1 (Pin_1), J2.2 (Pin_2), J2.3 (Pin_3), J2.4 (Pin_4), J2.5 (Pin_5), JP1.1 (Pin_1), JP1.2 (Pin_2), L1.1 (Pin_1), L1.2 (Pin_2), L2.1 (Pin_1), L2.2 (Pin_2), L2.3 (Pin_3), L2.4 (Pin_4), Q1.1 (Pin_1), Q1.2 (Pin_2), Q1.3 (Pin_3), Q1.4 (Pin_4), Q4.1 (Pin_1), Q4.2 (Pin_2), Q4.3 (Pin_3), Q4.4 (Pin_4), Q4.5 (Pin_5), Q4.6 (Pin_6), Q4.7 (Pin_7), Q4.8 (Pin_8), Q5.1 (Pin_1), Q5.2 (Pin_2), Q5.3 (Pin_3), Q5.4 (Pin_4), Q5.5 (Pin_5), Q5.6 (Pin_6), Q5.7 (Pin_7), Q5.8 (Pin_8), R1.1 (Pin_1), R1.2 (Pin_2), R10.1 (Pin_1), R10.2 (Pin_2), R101.1 (Pin_1), R101.2 (Pin_2), R102.1 (Pin_1), R102.2 (Pin_2), R103.1 (Pin_1), R103.2 (Pin_2), R104.1 (Pin_1), R104.2 (Pin_2), R105.1 (Pin_1), R105.2 (Pin_2), R106.1 (Pin_1), R106.2 (Pin_2), R107.2 (Pin_2), R108.1 (Pin_1), R108.2 (Pin_2), R111.1 (Pin_1), R111.2 (Pin_2), R112.1 (Pin_1), R112.2 (Pin_2), R113.1 (Pin_1), R113.2 (Pin_2), R114.1 (Pin_1), R114.2 (Pin_2), R115.1 (Pin_1), R115.2 (Pin_2), R116.1 (Pin_1), R116.2 (Pin_2), R117.1 (Pin_1), R117.2 (Pin_2), R118.1 (Pin_1), R118.2 (Pin_2), R2.1 (Pin_1), R3.1 (Pin_1), R3.2 (Pin_2), R4.1 (Pin_1), R4.2 (Pin_2), R5.1 (Pin_1), R5.2 (Pin_2), R6.1 (Pin_1), R6.2 (Pin_2), R7.1 (Pin_1), R7.2 (Pin_2), R8.1 (Pin_1), R8.2 (Pin_2), R9.1 (Pin_1), R9.2 (Pin_2), TP1.1 (Pin_1), TP2.1 (Pin_1), TP3.1 (Pin_1), TVS11.1 (Pin_1), TVS11.2 (Pin_2), TVS12.1 (Pin_1), TVS12.2 (Pin_2), TVS13.1 (Pin_1), TVS13.2 (Pin_2), TVS14.1 (Pin_1), TVS14.2 (Pin_2), TVS15.1 (Pin_1), TVS15.2 (Pin_2), TVS16.1 (Pin_1), TVS16.2 (Pin_2), TVS17.2 (Pin_2), TVS18.1 (Pin_1), TVS18.2 (Pin_2), U1.10 (Pin_10), U1.11 (Pin_11), U1.12 (Pin_12), U1.13 (Pin_13), U1.14 (Pin_14), U1.15 (Pin_15), U1.16 (Pin_16), U1.17 (Pin_17), U1.18 (Pin_18), U1.19 (Pin_19), U1.20 (Pin_20), U1.21 (Pin_21), U1.22 (Pin_22), U1.23 (Pin_23), U1.24 (Pin_24), U1.25 (Pin_25), U1.26 (Pin_26), U1.27 (Pin_27), U1.28 (Pin_28), U1.29 (Pin_29), U1.30 (Pin_30), U1.31 (Pin_31), U1.32 (Pin_32), U1.33 (Pin_33), U1.34 (Pin_34), U1.35 (Pin_35), U1.36 (Pin_36), U1.37 (Pin_37), U1.38 (Pin_38), U1.39 (Pin_39), U1.4 (Pin_4), U1.40 (Pin_40), U1.41 (Pin_41), U1.42 (Pin_42), U1.43 (Pin_43), U1.44 (Pin_44), U1.45 (Pin_45), U1.46 (Pin_46), U1.5 (Pin_5), U1.6 (Pin_6), U1.7 (Pin_7), U10.1 (Pin_1), U10.2 (Pin_2), U10.3 (Pin_3), U10.4 (Pin_4), U10.5 (Pin_5), U10.6 (Pin_6), U10.7 (Pin_7), U11.3 (Pin_3), U11.4 (Pin_4), U11.5 (Pin_5), U2.2 (Pin_2), U2.4 (Pin_4), U2.5 (Pin_5), U2.6 (Pin_6), U3.1 (Pin_1), U3.2 (Pin_2), U3.3 (Pin_3), U3.5 (Pin_5), U4.1 (Pin_1), U4.2 (Pin_2), U4.4 (Pin_4), U4.5 (Pin_5), U5.1 (Pin_1), U5.10 (Pin_10), U5.11 (Pin_11), U5.12 (Pin_12), U5.13 (Pin_13), U5.14 (Pin_14), U5.15 (Pin_15), U5.16 (Pin_16), U5.3 (Pin_3), U5.4 (Pin_4), U5.5 (Pin_5), U5.6 (Pin_6), U5.7 (Pin_7), U5.8 (Pin_8), U5.9 (Pin_9), U6.1 (Pin_1), U6.10 (Pin_10), U6.11 (Pin_11), U6.12 (Pin_12), U6.13 (Pin_13), U6.14 (Pin_14), U6.15 (Pin_15), U6.16 (Pin_16), U6.4 (Pin_4), U6.5 (Pin_5), U6.6 (Pin_6), U6.7 (Pin_7), U6.8 (Pin_8), U6.9 (Pin_9), U7.1 (Pin_1), U7.3 (Pin_3), U7.4 (Pin_4), U7.5 (Pin_5), U7.6 (Pin_6), U7.7 (Pin_7), U8.1 (Pin_1), U8.2 (Pin_2), U8.3 (Pin_3), U8.4 (Pin_4), U8.5 (Pin_5), U8.6 (Pin_6), U8.7 (Pin_7), U8.8 (Pin_8), U9.1 (Pin_1), U9.2 (Pin_2), U9.3 (Pin_3), U9.4 (Pin_4), U9.5 (Pin_5), U9.6 (Pin_6), U9.7 (Pin_7), U9.8 (Pin_8)
- net AIN7: now reaches J1.15 (Pin_15)
- net AIN7: now also R107.1 (Pin_1), TVS17.1 (Pin_1), U5.2 (Pin_2), U6.2 (Pin_2)
- net EXC_4K7: now reaches R2.2 (Pin_2)
- net EXC_4K7: now also U6.3 (Pin_3)
- net SENSOR_5V_OC: now reaches U4.3 (Pin_3)
- net BUCK_BOOT: now reaches U2.1 (Pin_1)
- net BUCK_FB: now reaches U2.3 (Pin_3)

Commit message: fix: complete CAN IO power monitor support circuits
Parts:
- added C10: 10nF 3V3 monitor filter, DIY_DASH:0603, symbol Connector_Generic:Conn_01x02
- added C11: 10nF IGN sense filter, DIY_DASH:0603, symbol Connector_Generic:Conn_01x02
- added C7: 100nF buck bootstrap, DIY_DASH:0603, symbol Connector_Generic:Conn_01x02
- added C8: 10nF VBAT monitor filter, DIY_DASH:0603, symbol Connector_Generic:Conn_01x02
- added C9: 10nF 5V monitor filter, DIY_DASH:0603, symbol Connector_Generic:Conn_01x02
- added R11: 40.2k 1% buck FB upper, DIY_DASH:0603, symbol Connector_Generic:Conn_01x02
- added R12: 10.0k 1% buck FB lower, DIY_DASH:0603, symbol Connector_Generic:Conn_01x02
- added R13: 100k 1% VBAT monitor upper, DIY_DASH:0603, symbol Connector_Generic:Conn_01x02
- added R14: 15.0k 1% VBAT monitor lower, DIY_DASH:0603, symbol Connector_Generic:Conn_01x02
- added R15: 10.0k 1% 5V monitor upper, DIY_DASH:0603, symbol Connector_Generic:Conn_01x02
- added R16: 18.0k 1% 5V monitor lower, DIY_DASH:0603, symbol Connector_Generic:Conn_01x02
- added R17: 1.00k 1% 3V3 monitor upper, DIY_DASH:0603, symbol Connector_Generic:Conn_01x02
- added R18: 100k 1% 3V3 monitor lower, DIY_DASH:0603, symbol Connector_Generic:Conn_01x02
- added R19: 100k 1% IGN sense upper, DIY_DASH:0603, symbol Connector_Generic:Conn_01x02
- added R20: 15.0k 1% IGN sense lower, DIY_DASH:0603, symbol Connector_Generic:Conn_01x02
Connections:
- net BUCK_BOOT is gone; now on net +3V3: U2.1 (Pin_1)
- net BUCK_FB is gone; now on net +3V3: U2.3 (Pin_3)
- net SENSOR_5V_OC is gone; now on net +3V3: U4.3 (Pin_3)
- net +3V3: now also U1.47 (Pin_47), C10.1 (Pin_1), C10.2 (Pin_2), C11.1 (Pin_1), C11.2 (Pin_2), C7.1 (Pin_1), C7.2 (Pin_2), C8.1 (Pin_1), C8.2 (Pin_2), C9.1 (Pin_1), C9.2 (Pin_2), R11.1 (Pin_1), R11.2 (Pin_2), R12.1 (Pin_1), R12.2 (Pin_2), R13.1 (Pin_1), R13.2 (Pin_2), R14.1 (Pin_1), R14.2 (Pin_2), R15.1 (Pin_1), R15.2 (Pin_2), R16.1 (Pin_1), R16.2 (Pin_2), R17.1 (Pin_1), R17.2 (Pin_2), R18.1 (Pin_1), R18.2 (Pin_2), R19.1 (Pin_1), R19.2 (Pin_2), R20.1 (Pin_1), R20.2 (Pin_2); no longer U1.37 (Pin_37)
Other:
- note added: "C10 / 0603"
- note added: "C11 / 0603"
- note added: "C7 / 0603"
- note added: "C8 / 0603"
- note added: "C9 / 0603"
- note added: "R11 / 0603"
- note added: "R12 / 0603"
- note added: "R13 / 0603"
- note added: "R14 / 0603"
- note added: "R15 / 0603"
- note added: "R16 / 0603"
- note added: "R17 / 0603"
- note added: "R18 / 0603"
- note added: "R19 / 0603"
- note added: "R20 / 0603"
