File: hardware/can-io-module/can-io-module.kicad_sch (KiCad schematic)
At the start: 95 parts, among them J1 ECU_FCI_24P_RightAngle, J2 SWD_1x05_P2.54mm_DNP, Q1 60V P-channel reverse polarity, Q4 60V logic N-MOS RELAY1, Q5 60V logic N-MOS RELAY2, U1 STM32G0B1CBT6, U10 MAX31855KASA+, U11 Schmitt Flex front end, U2 LMR16006Y-Q1, U3 3V3 LDO 300mA, U4 SENSOR_5V load switch, U5 74HCT4051 1K excitation, U6 74HCT4051 4K7 excitation, U7 L9613, U8 TJA1051T/3, U9 TLV9002-Q1

Commit message: fix: route schematic nets without crossing component pins
Connections:
- net +3V3: no longer C1.1 (Pin_1), C1.2 (Pin_2), C10.1 (Pin_1), C10.2 (Pin_2), C101.1 (Pin_1), C101.2 (Pin_2), C102.1 (Pin_1), C102.2 (Pin_2), C103.1 (Pin_1), C103.2 (Pin_2), C104.1 (Pin_1), C104.2 (Pin_2), C105.1 (Pin_1), C105.2 (Pin_2), C106.1 (Pin_1), C106.2 (Pin_2), C107.1 (Pin_1), C107.2 (Pin_2), C108.1 (Pin_1), C108.2 (Pin_2), C11.1 (Pin_1), C11.2 (Pin_2), C2.1 (Pin_1), C2.2 (Pin_2), C3.2 (Pin_2), C4.2 (Pin_2), C5.2 (Pin_2), C6.1 (Pin_1), C6.2 (Pin_2), C7.1 (Pin_1), C7.2 (Pin_2), C8.1 (Pin_1), C8.2 (Pin_2), C9.1 (Pin_1), C9.2 (Pin_2), D1.1 (Pin_1), D1.2 (Pin_2), D2.1 (Pin_1), D2.2 (Pin_2), D3.1 (Pin_1), D3.2 (Pin_2), D4.1 (Pin_1), D4.2 (Pin_2), D5.1 (Pin_1), D5.2 (Pin_2), D6.1 (Pin_1), D6.2 (Pin_2), D7.1 (Pin_1), D7.2 (Pin_2), F1.1 (Pin_1), F1.2 (Pin_2), F2.1 (Pin_1), F2.2 (Pin_2), FB1.2 (Pin_2), J1.1 (Pin_1), J1.10 (Pin_10), J1.11 (Pin_11), J1.12 (Pin_12), J1.13 (Pin_13), J1.14 (Pin_14), J1.16 (Pin_16), J1.17 (Pin_17), J1.18 (Pin_18), J1.19 (Pin_19), J1.2 (Pin_2), J1.20 (Pin_20), J1.21 (Pin_21), J1.22 (Pin_22), J1.23 (Pin_23), J1.24 (Pin_24), J1.3 (Pin_3), J1.4 (Pin_4), J1.5 (Pin_5), J1.6 (Pin_6), J1.7 (Pin_7), J1.8 (Pin_8), J1.9 (Pin_9), J2.2 (Pin_2), J2.3 (Pin_3), J2.4 (Pin_4), J2.5 (Pin_5), JP1.1 (Pin_1), JP1.2 (Pin_2), L1.1 (Pin_1), L1.2 (Pin_2), L2.1 (Pin_1), L2.2 (Pin_2), L2.3 (Pin_3), L2.4 (Pin_4), Q1.1 (Pin_1), Q1.2 (Pin_2), Q1.3 (Pin_3), Q1.4 (Pin_4), Q4.1 (Pin_1), Q4.2 (Pin_2), Q4.3 (Pin_3), Q4.4 (Pin_4), Q4.5 (Pin_5), Q4.6 (Pin_6), Q4.7 (Pin_7), Q4.8 (Pin_8), Q5.1 (Pin_1), Q5.2 (Pin_2), Q5.3 (Pin_3), Q5.4 (Pin_4), Q5.5 (Pin_5), Q5.6 (Pin_6), Q5.7 (Pin_7), Q5.8 (Pin_8), R1.1 (Pin_1), R1.2 (Pin_2), R10.1 (Pin_1), R10.2 (Pin_2), R101.1 (Pin_1), R101.2 (Pin_2), R102.1 (Pin_1), R102.2 (Pin_2), R103.1 (Pin_1), R103.2 (Pin_2), R104.1 (Pin_1), R104.2 (Pin_2), R105.1 (Pin_1), R105.2 (Pin_2), R106.1 (Pin_1), R106.2 (Pin_2), R107.2 (Pin_2), R108.1 (Pin_1), R108.2 (Pin_2), R11.1 (Pin_1), R11.2 (Pin_2), R111.1 (Pin_1), R111.2 (Pin_2), R112.1 (Pin_1), R112.2 (Pin_2), R113.1 (Pin_1), R113.2 (Pin_2), R114.1 (Pin_1), R114.2 (Pin_2), R115.1 (Pin_1), R115.2 (Pin_2), R116.1 (Pin_1), R116.2 (Pin_2), R117.1 (Pin_1), R117.2 (Pin_2), R118.1 (Pin_1), R118.2 (Pin_2), R12.1 (Pin_1), R12.2 (Pin_2), R13.1 (Pin_1), R13.2 (Pin_2), R14.1 (Pin_1), R14.2 (Pin_2), R15.1 (Pin_1), R15.2 (Pin_2), R16.1 (Pin_1), R16.2 (Pin_2), R17.2 (Pin_2), R18.1 (Pin_1), R18.2 (Pin_2), R19.1 (Pin_1), R19.2 (Pin_2), R2.1 (Pin_1), R20.1 (Pin_1), R20.2 (Pin_2), R3.1 (Pin_1), R3.2 (Pin_2), R4.1 (Pin_1), R4.2 (Pin_2), R5.1 (Pin_1), R5.2 (Pin_2), R6.1 (Pin_1), R6.2 (Pin_2), R7.1 (Pin_1), R7.2 (Pin_2), R8.1 (Pin_1), R8.2 (Pin_2), R9.2 (Pin_2), TP1.1 (Pin_1), TP2.1 (Pin_1), TP3.1 (Pin_1), TVS11.1 (Pin_1), TVS11.2 (Pin_2), TVS12.1 (Pin_1), TVS12.2 (Pin_2), TVS13.1 (Pin_1), TVS13.2 (Pin_2), TVS14.1 (Pin_1), TVS14.2 (Pin_2), TVS15.1 (Pin_1), TVS15.2 (Pin_2), TVS16.1 (Pin_1), TVS16.2 (Pin_2), TVS17.2 (Pin_2), TVS18.1 (Pin_1), TVS18.2 (Pin_2), U1.10 (Pin_10), U1.11 (Pin_11), U1.12 (Pin_12), U1.13 (Pin_13), U1.14 (Pin_14), U1.15 (Pin_15), U1.16 (Pin_16), U1.17 (Pin_17), U1.18 (Pin_18), U1.19 (Pin_19), U1.20 (Pin_20), U1.21 (Pin_21), U1.22 (Pin_22), U1.23 (Pin_23), U1.24 (Pin_24), U1.25 (Pin_25), U1.26 (Pin_26), U1.27 (Pin_27), U1.28 (Pin_28), U1.29 (Pin_29), U1.30 (Pin_30), U1.31 (Pin_31), U1.32 (Pin_32), U1.33 (Pin_33), U1.34 (Pin_34), U1.35 (Pin_35), U1.36 (Pin_36), U1.38 (Pin_38), U1.39 (Pin_39), U1.40 (Pin_40), U1.41 (Pin_41), U1.42 (Pin_42), U1.43 (Pin_43), U1.44 (Pin_44), U1.45 (Pin_45), U1.46 (Pin_46), U1.47 (Pin_47), U1.5 (Pin_5), U1.7 (Pin_7), U10.1 (Pin_1), U10.2 (Pin_2), U10.3 (Pin_3), U10.5 (Pin_5), U10.6 (Pin_6), U10.7 (Pin_7), U11.2 (Pin_2), U11.3 (Pin_3), U11.4 (Pin_4), U2.1 (Pin_1), U2.2 (Pin_2), U2.3 (Pin_3), U2.4 (Pin_4), U2.5 (Pin_5), U2.6 (Pin_6), U3.1 (Pin_1), U3.2 (Pin_2), U3.3 (Pin_3), U4.1 (Pin_1), U4.2 (Pin_2), U4.3 (Pin_3), U4.4 (Pin_4), U4.5 (Pin_5), U5.1 (Pin_1), U5.10 (Pin_10), U5.11 (Pin_11), U5.12 (Pin_12), U5.13 (Pin_13), U5.14 (Pin_14), U5.15 (Pin_15), U5.16 (Pin_16), U5.3 (Pin_3), U5.4 (Pin_4), U5.5 (Pin_5), U5.6 (Pin_6), U5.7 (Pin_7), U5.8 (Pin_8), U5.9 (Pin_9), U6.1 (Pin_1), U6.10 (Pin_10), U6.11 (Pin_11), U6.12 (Pin_12), U6.13 (Pin_13), U6.14 (Pin_14), U6.15 (Pin_15), U6.16 (Pin_16), U6.4 (Pin_4), U6.5 (Pin_5), U6.6 (Pin_6), U6.7 (Pin_7), U6.8 (Pin_8), U6.9 (Pin_9), U7.1 (Pin_1), U7.3 (Pin_3), U7.4 (Pin_4), U7.5 (Pin_5), U7.6 (Pin_6), U7.7 (Pin_7), U8.1 (Pin_1), U8.2 (Pin_2), U8.3 (Pin_3), U8.4 (Pin_4), U8.6 (Pin_6), U8.7 (Pin_7), U8.8 (Pin_8), U9.1 (Pin_1), U9.2 (Pin_2), U9.3 (Pin_3), U9.4 (Pin_4), U9.5 (Pin_5), U9.6 (Pin_6), U9.7 (Pin_7), U9.8 (Pin_8)
- new net +5V: C2.1 (Pin_1), L1.2 (Pin_2), R1.1 (Pin_1), R11.1 (Pin_1), R15.1 (Pin_1), R2.1 (Pin_1), R3.1 (Pin_1), R4.1 (Pin_1), U3.1 (Pin_1), U3.3 (Pin_3), U4.5 (Pin_5), U5.16 (Pin_16), U6.16 (Pin_16), U7.3 (Pin_3), U8.3 (Pin_3), U9.8 (Pin_8)
- new net ADC_IN1: C101.1 (Pin_1), R101.2 (Pin_2), R111.1 (Pin_1), U1.11 (Pin_11)
- new net ADC_IN2: C102.1 (Pin_1), R102.2 (Pin_2), R112.1 (Pin_1), U1.12 (Pin_12)
- new net ADC_IN3: C103.1 (Pin_1), R103.2 (Pin_2), R113.1 (Pin_1), U1.13 (Pin_13)
- new net ADC_IN4: C104.1 (Pin_1), R104.2 (Pin_2), R114.1 (Pin_1), U1.14 (Pin_14)
- new net ADC_IN5: C105.1 (Pin_1), R105.2 (Pin_2), R115.1 (Pin_1), U1.17 (Pin_17)
- new net ADC_IN6: C106.1 (Pin_1), R106.2 (Pin_2), R116.1 (Pin_1), U1.18 (Pin_18)
- new net ADC_IN7: C107.1 (Pin_1), R107.2 (Pin_2), R117.1 (Pin_1), U1.19 (Pin_19)
- new net ADC_IN8: C108.1 (Pin_1), R108.2 (Pin_2), R118.1 (Pin_1), U1.20 (Pin_20)
- new net AIN1: J1.9 (Pin_9), R101.1 (Pin_1), TVS11.1 (Pin_1), U5.13 (Pin_13), U6.13 (Pin_13)
- new net AIN2: J1.10 (Pin_10), R102.1 (Pin_1), TVS12.1 (Pin_1), U5.14 (Pin_14), U6.14 (Pin_14)
- new net AIN3: J1.11 (Pin_11), R103.1 (Pin_1), TVS13.1 (Pin_1), U5.15 (Pin_15), U6.15 (Pin_15)
- new net AIN4: J1.12 (Pin_12), R104.1 (Pin_1), TVS14.1 (Pin_1), U5.12 (Pin_12), U6.12 (Pin_12)
- new net AIN5: J1.13 (Pin_13), R105.1 (Pin_1), TVS15.1 (Pin_1), U5.1 (Pin_1), U6.1 (Pin_1)
- new net AIN6: J1.14 (Pin_14), R106.1 (Pin_1), TVS16.1 (Pin_1), U5.5 (Pin_5), U6.5 (Pin_5)
- new net AIN8: J1.16 (Pin_16), R108.1 (Pin_1), TVS18.1 (Pin_1), U5.4 (Pin_4), U6.4 (Pin_4)
- new net AOUT1: D6.1 (Pin_1), J1.22 (Pin_22), R7.2 (Pin_2)
- new net AOUT1_OP: R7.1 (Pin_1), U9.2 (Pin_2), U9.3 (Pin_3)
- new net AOUT2: D7.1 (Pin_1), J1.23 (Pin_23), R8.2 (Pin_2)
- new net AOUT2_OP: R8.1 (Pin_1), U9.6 (Pin_6), U9.7 (Pin_7)
- new net BOOT0: R10.1 (Pin_1), U1.21 (Pin_21)
- new net BUCK_BOOT: C7.1 (Pin_1), U2.1 (Pin_1)
- new net BUCK_FB: R11.2 (Pin_2), R12.1 (Pin_1), U2.3 (Pin_3)
- new net BUCK_SW: C7.2 (Pin_2), D2.2 (Pin_2), L1.1 (Pin_1), U2.6 (Pin_6)
- new net CAN_H: D3.1 (Pin_1), J1.4 (Pin_4), JP1.1 (Pin_1), L2.3 (Pin_3)
- new net CAN_H_PROTECTED: L2.1 (Pin_1), U8.7 (Pin_7)
- new net CAN_L: D3.2 (Pin_2), J1.5 (Pin_5), JP1.2 (Pin_2), L2.4 (Pin_4)
- new net CAN_L_PROTECTED: L2.2 (Pin_2), U8.6 (Pin_6)
- new net CAN_RX: U1.33 (Pin_33), U8.4 (Pin_4)
- new net CAN_SILENT: U1.26 (Pin_26), U8.8 (Pin_8)
- new net CAN_TX: U1.34 (Pin_34), U8.1 (Pin_1)
- new net DAC1_RAW: U1.15 (Pin_15), U9.1 (Pin_1)
- new net DAC2_RAW: U1.16 (Pin_16), U9.5 (Pin_5)
- new net EGT_CS: U1.44 (Pin_44), U10.6 (Pin_6)
- new net EGT_K_NEG: J1.18 (Pin_18), U10.3 (Pin_3)
- new net EGT_K_POS: J1.17 (Pin_17), U10.2 (Pin_2)
- new net EGT_SCK: U1.42 (Pin_42), U10.5 (Pin_5)
- new net EGT_SO: U1.43 (Pin_43), U10.7 (Pin_7)
- new net EXC_1K: R1.2 (Pin_2), U5.3 (Pin_3)
- new net FLEX_CAPTURE: U1.28 (Pin_28), U11.4 (Pin_4)
- new net FLEX_IN: D5.1 (Pin_1), J1.21 (Pin_21), U11.2 (Pin_2)
- new net IGN: J1.3 (Pin_3), Q1.1 (Pin_1), R19.1 (Pin_1), U2.4 (Pin_4)
- new net IGN_SENSE: C11.1 (Pin_1), R19.2 (Pin_2), R20.1 (Pin_1), U1.29 (Pin_29)
- new net KRX: U1.46 (Pin_46), U7.1 (Pin_1)
- new net KTX: U1.45 (Pin_45), U7.4 (Pin_4)
- new net K_LINE: D4.1 (Pin_1), J1.6 (Pin_6), U7.6 (Pin_6)
- new net NRST: J2.4 (Pin_4), R9.2 (Pin_2), TP3.1 (Pin_1), U1.10 (Pin_10)
- new net POWER_GND: C1.2 (Pin_2), C10.2 (Pin_2), C11.2 (Pin_2), C2.2 (Pin_2), C3.2 (Pin_2), C4.2 (Pin_2), C5.2 (Pin_2), C6.2 (Pin_2), C8.2 (Pin_2), C9.2 (Pin_2), D1.2 (Pin_2), D2.1 (Pin_1), D4.2 (Pin_2), D5.2 (Pin_2), D6.2 (Pin_2), D7.2 (Pin_2), J1.2 (Pin_2), J2.5 (Pin_5), Q4.3 (Pin_3), Q5.3 (Pin_3), R10.2 (Pin_2), R12.2 (Pin_2), R14.2 (Pin_2), R16.2 (Pin_2), R18.2 (Pin_2), R20.2 (Pin_2), R5.2 (Pin_2), R6.2 (Pin_2), TVS11.2 (Pin_2), TVS12.2 (Pin_2), TVS13.2 (Pin_2), TVS14.2 (Pin_2), TVS15.2 (Pin_2), TVS16.2 (Pin_2), TVS17.2 (Pin_2), TVS18.2 (Pin_2), U1.7 (Pin_7), U10.1 (Pin_1), U11.3 (Pin_3), U2.2 (Pin_2), U3.2 (Pin_2), U4.2 (Pin_2), U5.7 (Pin_7), U5.8 (Pin_8), U6.7 (Pin_7), U6.8 (Pin_8), U7.5 (Pin_5), U8.2 (Pin_2), U9.4 (Pin_4)
- new net PULL_1K_EN_N: R3.2 (Pin_2), U1.41 (Pin_41), U5.6 (Pin_6)
- new net PULL_4K7_EN_N: R4.2 (Pin_2), U1.30 (Pin_30), U6.6 (Pin_6)
- new net PULL_A0: U1.38 (Pin_38), U5.11 (Pin_11), U6.11 (Pin_11)
- new net PULL_A1: U1.39 (Pin_39), U5.10 (Pin_10), U6.10 (Pin_10)
- new net PULL_A2: U1.40 (Pin_40), U5.9 (Pin_9), U6.9 (Pin_9)
- new net RELAY1_GATE: Q4.1 (Pin_1), R5.1 (Pin_1), U1.31 (Pin_31)
- new net RELAY2_GATE: Q5.1 (Pin_1), R6.1 (Pin_1), U1.25 (Pin_25)
- new net RELAY_OUT1: J1.19 (Pin_19), Q4.2 (Pin_2), Q4.4 (Pin_4), Q4.5 (Pin_5), Q4.6 (Pin_6), Q4.7 (Pin_7), Q4.8 (Pin_8)
- new net RELAY_OUT2: J1.20 (Pin_20), Q5.2 (Pin_2), Q5.4 (Pin_4), Q5.5 (Pin_5), Q5.6 (Pin_6), Q5.7 (Pin_7), Q5.8 (Pin_8)
- new net SENSOR_5V: F2.2 (Pin_2), J1.7 (Pin_7)
- new net SENSOR_5V_EN: U1.27 (Pin_27), U4.4 (Pin_4)
- new net SENSOR_5V_OC: U1.47 (Pin_47), U4.3 (Pin_3)
- new net SENSOR_5V_SW: F2.1 (Pin_1), U4.1 (Pin_1)
- new net SENSOR_GND: C101.2 (Pin_2), C102.2 (Pin_2), C103.2 (Pin_2), C104.2 (Pin_2), C105.2 (Pin_2), C106.2 (Pin_2), C107.2 (Pin_2), C108.2 (Pin_2), J1.8 (Pin_8), R111.2 (Pin_2), R112.2 (Pin_2), R113.2 (Pin_2), R114.2 (Pin_2), R115.2 (Pin_2), R116.2 (Pin_2), R117.2 (Pin_2), R118.2 (Pin_2)
- new net SERVICE: J1.24 (Pin_24), U1.32 (Pin_32)
- new net SWCLK: J2.3 (Pin_3), TP2.1 (Pin_1), U1.36 (Pin_36)
- new net SWDIO: J2.2 (Pin_2), TP1.1 (Pin_1), U1.35 (Pin_35)
- new net V3V3_MON: C10.1 (Pin_1), R17.2 (Pin_2), R18.1 (Pin_1), U1.24 (Pin_24)
- new net V5_MON: C9.1 (Pin_1), R15.2 (Pin_2), R16.1 (Pin_1), U1.23 (Pin_23)
- new net VBAT: F1.1 (Pin_1), J1.1 (Pin_1)
- new net VBAT_FUSED: F1.2 (Pin_2), Q1.3 (Pin_3), Q1.4 (Pin_4)
- new net VBAT_MON: C8.1 (Pin_1), R13.2 (Pin_2), R14.1 (Pin_1), U1.22 (Pin_22)
- new net VBAT_PROTECTED: C1.1 (Pin_1), D1.1 (Pin_1), Q1.2 (Pin_2), R13.1 (Pin_1), U2.5 (Pin_5), U7.7 (Pin_7)
- new net VDDA: C6.1 (Pin_1), FB1.2 (Pin_2), U1.5 (Pin_5)
